File: pcb/driveboard.sch (KiCad schematic (older format))
At the start: 49 parts, among them IC1 7411, IC2 7410, P1 AC IN, P2 AC out, P3 5V in, P6 AQV2526, x1 RJ45, x2 RJ45, y1 RJ45, y2 RJ45

Commit message: Bugfix: Change R1-R9 from pullups to pulldowns.
Connections:
- net GND: now also R1.2, R2.2, R3.2, R4.2, R5.1, R6.1, R7.2, R8.2, R9.2
- net at C10.1, C9.1, IC1.14 (VDD)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: no longer Arduino1.4 (P4), IC1.9 (3A), R1.1, R2.1, R3.1, R4.2, R5.1, R6.1, R7.1, R8.1, R9.1
- net at Arduino1.6 (P6), IC1.3 (2A), y1.2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: now also R3.1; no longer R3.2
- net at Arduino1.7 (P7), IC1.4 (2B), x2.2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: now also R1.1; no longer R2.2
- net at Arduino1.8 (P8), IC1.5 (2C), x1.2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: now also R2.1; no longer R1.2
- net at IC1.10 (3B), door1.2, door1.4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: now also R9.1; no longer R9.2
- net at IC1.11 (3C), door2.2, door2.4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: now also R8.1; no longer R8.2
- net at Arduino2.6 (P6), IC2.11 (3C), chiller1.2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: now also R7.1; no longer R7.2
- new net: Arduino1.4 (P4), IC1.9 (3A)
Other:
- moved on the sheet: R1, R2, R3, R7, R8, R9
Changed lines of the file:
@@
 L R R3
 U 1 1 554BD7D2
-P 6450 2650
-F 0 "R3" V 6530 2650 40  0000 C CNN
-F 1 "10K" V 6457 2651 40  0000 C CNN
-F 2 "Resistors_SMD:R_0603" V 6380 2650 30  0001 C CNN
-F 3 "" H 6450 2650 30  0000 C CNN
-	1    6450 2650
+P 6250 3550
+F 0 "R3" V 6330 3550 40  0000 C CNN
+F 1 "10K" V 6257 3551 40  0000 C CNN
+F 2 "Resistors_SMD:R_0603" V 6180 3550 30  0001 C CNN
+F 3 "" H 6250 3550 30  0000 C CNN
+	1    6250 3550
 	1    0    0    -1
 $EndComp
@@
 L R R2
 U 1 1 554BD804
-P 6950 2650
-F 0 "R2" V 7030 2650 40  0000 C CNN
-F 1 "10K" V 6957 2651 40  0000 C CNN
-F 2 "Resistors_SMD:R_0603" V 6880 2650 30  0001 C CNN
-F 3 "" H 6950 2650 30  0000 C CNN
-	1    6950 2650
+P 6050 3550
+F 0 "R2" V 6130 3550 40  0000 C CNN
+F 1 "10K" V 6057 3551 40  0000 C CNN
+F 2 "Resistors_SMD:R_0603" V 5980 3550 30  0001 C CNN
+F 3 "" H 6050 3550 30  0000 C CNN
+	1    6050 3550
 	1    0    0    -1
 $EndComp
@@
 L R R1
 U 1 1 554BD829
-P 6700 2650
-F 0 "R1" V 6780 2650 40  0000 C CNN
-F 1 "10K" V 6707 2651 40  0000 C CNN
-F 2 "Resistors_SMD:R_0603" V 6630 2650 30  0001 C CNN
-F 3 "" H 6700 2650 30  0000 C CNN
-	1    6700 2650
+P 6450 3550
+F 0 "R1" V 6530 3550 40  0000 C CNN
+F 1 "10K" V 6457 3551 40  0000 C CNN
+F 2 "Resistors_SMD:R_0603" V 6380 3550 30  0001 C CNN
+F 3 "" H 6450 3550 30  0000 C CNN
+	1    6450 3550
 	1    0    0    -1
 $EndComp
@@
 L R R8
 U 1 1 554C08F0
-P 5350 5350
-F 0 "R8" V 5430 5350 40  0000 C CNN
-F 1 "10K" V 5357 5351 40  0000 C CNN
-F 2 "Resistors_SMD:R_0603" V 5280 5350 30  0001 C CNN
-F 3 "" H 5350 5350 30  0000 C CNN
-	1    5350 5350
+P 5350 5850
+F 0 "R8" V 5430 5850 40  0000 C CNN
+F 1 "10K" V 5357 5851 40  0000 C CNN
+F 2 "Resistors_SMD:R_0603" V 5280 5850 30  0001 C CNN
+F 3 "" H 5350 5850 30  0000 C CNN
+	1    5350 5850
 	1    0    0    -1
 $EndComp
@@
 L R R9
 U 1 1 554C0934
-P 4750 5350
-F 0 "R9" V 4830 5350 40  0000 C CNN
-F 1 "10K" V 4757 5351 40  0000 C CNN
-F 2 "Resistors_SMD:R_0603" V 4680 5350 30  0001 C CNN
-F 3 "" H 4750 5350 30  0000 C CNN
-	1    4750 5350
+P 5100 5850
+F 0 "R9" V 5180 5850 40  0000 C CNN
+F 1 "10K" V 5107 5851 40  0000 C CNN
+F 2 "Resistors_SMD:R_0603" V 5030 5850 30  0001 C CNN
+F 3 "" H 5100 5850 30  0000 C CNN
+	1    5100 5850
 	1    0    0    -1
 $EndComp
@@
 L R R7
 U 1 1 55606132
-P 12200 5950
-F 0 "R7" V 12280 5950 50  0000 C CNN
-F 1 "10K" V 12200 5950 50  0000 C CNN
-F 2 "Resistors_SMD:R_0603" V 12130 5950 30  0001 C CNN
-F 3 "" H 12200 5950 30  0000 C CNN
-	1    12200 5950
+P 12500 5800
+F 0 "R7" V 12580 5800 50  0000 C CNN
+F 1 "10K" V 12500 5800 50  0000 C CNN
+F 2 "Resistors_SMD:R_0603" V 12430 5800 30  0001 C CNN
+F 3 "" H 12500 5800 30  0000 C CNN
+	1    12500 5800
 	1    0    0    -1
 $EndComp
@@
 	6950 3300 8800 3300
 Wire Wire Line
-	6950 2800 6950 3600
+	6950 3000 6950 3600
 Wire Wire Line
 	8500 3300 8500 3700
@@
 	6100 5600 4750 5600
 Wire Wire Line
-	4750 5500 4750 7050
-Wire Wire Line
 	4350 6350 4750 6350
 Wire Wire Line
@@
 Connection ~ 5350 7050
 Wire Wire Line
-	4750 2650 4750 5200
-Wire Wire Line
 	4750 2650 4900 2650
-Connection ~ 4750 5100
 Wire Wire Line
 	7950 3600 7950 4150
@@
 Wire Wire Line
 	3900 3300 4750 3300
-Connection ~ 4750 3300
 Wire Wire Line
 	3900 3200 5900 3200
@@
 	6950 3600 7350 3600
 Wire Wire Line
-	6950 2500 6950 2150
-Connection ~ 6950 2150
-Connection ~ 6950 3000
-Wire Wire Line
 	3900 2900 6700 2900
 Wire Wire Line
-	6700 2800 6700 3700
-Connection ~ 6700 2900
-Wire Wire Line
-	6700 2500 6700 2150
-Connection ~ 6700 2150
-Wire Wire Line
-	6450 2800 6450 3100
-Connection ~ 6450 3100
-Wire Wire Line
-	6450 2500 6450 2150
-Connection ~ 6450 2150
+	6700 2900 6700 3700
 Wire Wire Line
 	5350 4350 7150 4350
@@
 	6700 4700 6700 5600
 Connection ~ 6700 5600
-Connection ~ 4750 5600
 Wire Wire Line
 	5850 5100 5850 5500
 Wire Wire Line
 	5850 5500 6100 5500
-Wire Wire Line
-	5350 5200 5350 5100
-Connection ~ 5350 5100
 Connection ~ 4150 7050
 Wire Wire Line
@@
 Connection ~ 5350 4250
 Wire Wire Line
-	4750 3800 5550 3800
-Connection ~ 4750 3800
-Connection ~ 5350 3800
-Wire Wire Line
 	11400 5100 11400 5150
 Wire Wire Line
@@
 Wire Wire Line
 	11750 4750 11750 4800
-Wire Wire Line
-	5350 5500 5350 5700
 Connection ~ 5850 5700
 Connection ~ 8800 6000
@@
 Wire Wire Line
 	3900 4800 4400 4800
-Wire Wire Line
-	12200 5800 12200 3750
-Connection ~ 12200 3750
-Connection ~ 12200 6100
 Wire Wire Line
 	3900 4700 6700 4700
@@
 	3550 6000 3550 5950
 Wire Wire Line
-	3650 5500 3100 5500
+	3100 5500 3650 5500
 Wire Wire Line
 	3550 5500 3550 5650
 Connection ~ 3550 5500
+Wire Wire Line
+	5350 3800 6450 3800
+Wire Wire Line
+	5800 3800 5800 3900
+$Comp
+L GND #PWR?
+U 1 1 55B0E9D4
+P 5800 3900
+F 0 "#PWR?" H 5800 3650 50  0001 C CNN
+F 1 "GND" H 5800 3750 50  0000 C CNN
+F 2 "" H 5800 3900 60  0000 C CNN
+F 3 "" H 5800 3900 60  0000 C CNN
+	1    5800 3900
+	1    0    0    -1
+$EndComp
+Wire Wire Line
+	6050 3400 6050 2900
+Connection ~ 6050 2900
+Wire Wire Line
+	6250 3400 6250 3100
+Connection ~ 6250 3100
+Wire Wire Line
+	6450 3400 6450 3000
+Connection ~ 6450 3000
+Wire Wire Line
+	6450 3800 6450 3700
+Connection ~ 5800 3800
+Wire Wire Line
+	6050 3700 6050 3800
+Connection ~ 6050 3800
+Wire Wire Line
+	6250 3700 6250 3800
+Connection ~ 6250 3800
+Wire Wire Line
+	5100 5700 5100 5600
+Connection ~ 5100 5600
+Wire Wire Line
+	4750 5600 4750 7050
+Wire Wire Line
+	4750 3300 4750 5100
+$Comp
+L GND #PWR?
+U 1 1 55B1536C
+P 5100 6000
+F 0 "#PWR?" H 5100 5750 50  0001 C CNN
+F 1 "GND" H 5100 5850 50  0000 C CNN
+F 2 "" H 5100 6000 60  0000 C CNN
+F 3 "" H 5100 6000 60  0000 C CNN
+	1    5100 6000
+	1    0    0    -1
+$EndComp
+Wire Wire Line
+	5100 6000 5350 6000
+Connection ~ 5100 6000
+Wire Wire Line
+	12500 5650 12350 5650
+Connection ~ 12350 5650
+$Comp
+L GND #PWR?
+U 1 1 55B1611D
+P 12500 5950
+F 0 "#PWR?" H 12500 5700 50  0001 C CNN
+F 1 "GND" H 12500 5800 50  0000 C CNN
+F 2 "" H 12500 5950 60  0000 C CNN
+F 3 "" H 12500 5950 60  0000 C CNN
+	1    12500 5950
+	1    0    0    -1
+$EndComp
 $EndSCHEMATC

Commit message: Re-add Vcc connection.
Connections:
- net at C10.1, C9.1, IC1.14 (VDD)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: now also Arduino1.4 (P4), C3.1, C4.1, IC1.9 (3A), P3.2 (P2), R17.1, SSR1.3
Changed lines of the file:
@@
 $EndComp
 Wire Wire Line
-	4900 2650 4900 2150
+	4900 3300 4900 2150
 Wire Wire Line
 	4900 2150 8800 2150
@@
 	7800 5150 11750 5150
 Wire Wire Line
-	6100 5600 4750 5600
+	4750 5600 6100 5600
 Wire Wire Line
 	4350 6350 4750 6350
@@
 	5050 7050 5350 7050
 Connection ~ 5350 7050
-Wire Wire Line
-	4750 2650 4900 2650
 Wire Wire Line
 	7950 3600 7950 4150
@@
 	4000 3500 4000 3700
 Wire Wire Line
-	3900 3300 4750 3300
+	3900 3300 4900 3300
 Wire Wire Line
 	3900 3200 5900 3200
@@
 	2350 9150 4550 9150
 Wire Wire Line
-	3400 9150 3400 9600
+	3400 6100 3400 9600
 Wire Wire Line
 	4250 8650 4250 10500
@@
 	4750 5600 4750 7050
 Wire Wire Line
-	4750 3300 4750 5100
+	4750 3300 4750 5500
 $Comp
 L GND #PWR?
@@
 	1    0    0    -1
 $EndComp
+Connection ~ 4750 3300
+Wire Wire Line
+	4750 5500 4600 5500
+Wire Wire Line
+	4600 5500 4600 6100
+Wire Wire Line
+	4600 6100 3400 6100
+Connection ~ 4750 5100
 $EndSCHEMATC
