File: pcb/lpcsaur/lpcsaur.sch (KiCad schematic (older format))
At the start: 163 parts, among them J1 X1, J2 X2, J3 Y1, J5 Z2, J6 Z2, J7 DOOR1, J8 DOOR2, U10 MICRO-SD, U6 LPC1768_TQFP100, X1 CRYSTAL 12MHz, Y2 Z1

Commit message: All components placed.
Parts:
- removed P?: CONN_01X03, symbol CONN_01X03
- added C16, C17: 10u, symbol CP
- added D1, D2: 1N5822, symbol D
- added J17, J19: RELAY1, symbol CONN_01X02
- added J18, J20: V-SELECT, symbol CONN_01X03
- added J23: SERIAL, symbol CONN_01X04
- added LED8, LED9: LED, symbol Led_Small
- added Q1, Q2: ZXMN4A06, symbol Q_NMOS_GDS
- added R24, R27: 10K, symbol R
- added R25, R28: 22, symbol R
- added R26, R29: 5K6, symbol R
- added R39: 10k, ~, symbol R
- added SW?: SW_PUSH, symbol SW_PUSH
- C1, C2, C3, C4, C5, C6, C7, C8: renamed from C?; value C -> 100n
- gave numbers to parts that had none: 43
- renumbered R28 to R37, R1 to R38, R27 to R40
Connections:
- net labels added: +24V, P1.0, P1.1, RESET
- net labels removed: P??
- wire segments 265 -> 299
- no-connect marks 20 -> 18

Commit message: Annotate.
Parts:
- removed C22, C23, C28, C29, C30, C31, C44, C45, C46, C6: 100n, ~, symbol C
- removed C24, C25, C26, C27: 100uF, ~, symbol CP
- removed W? (x8): TEST_1P, symbol TEST_1P
- removed X1: CRYSTAL 12MHz, symbol CRYSTAL_SMD
- added C32: 100n, ~, symbol C
- added C33: 10u, symbol CP
- added C34, C35: 100u, symbol CP
- added J25: 12V IN, symbol CONN_01X02
- added J26: 24V IN, symbol CONN_01X02
- added J27: AUX I/O, symbol CONN_01X10
- added X1: CRYSTAL, symbol CRYSTAL
- C28: renamed from C?; value CP -> 10u
- C29: renamed from C?; value C -> 100n
- D3, D4: renamed from D?; value D -> MBRA210LT3
- IC3: renamed from U?; value 7408 -> 74HCT08
- J10: value Laser control -> LASER
- J24: renamed from P?; value CONN_01X02 -> 5V IN
- J28: renamed from chiller?; value CONN_01X02 -> CHILLER
- J9: value e-stop -> E-STOP
- L1: value INDUCTOR -> 39 nH
- gave numbers to parts that had none: 19
- renumbered C11 to C20, C12 to C21, C13 to C22, C14 to C23, C15 to C24, C16 to C25, C17 to C26, C1 to C27, C20 to C30, C21 to C31, C18 to C36, C19 to C37, LED8 to LED10, LED9 to LED11, D6 to LED8, R41 to R42, R42 to R43, R43 to R44, R17 to R45, R18 to R46
Connections:
- net labels removed: +5VD, RESET, STP1, STP2, STP3, STP4
- wire segments 299 -> 327
Other:
- note added: "Located near VDD"
- moved on the sheet: C14, C15, C20, C21, C22, C23, C24, C25, C28, C29, C30, C31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

Commit message: Make ERC pass.
Parts:
- LED10: value LED -> SSR1
- LED11: value LED -> SSR2
- LED7: value disable -> Disable
- LED8: value LED -> Play
- LED9: value LED -> 3V3
- R38, R39, R40, R42, R43, R44: value 10k -> 10K
- X1: value CRYSTAL -> 12 MHz
- renumbered U6 to IC7, U10 to J29, W4 to JTAG1, W5 to JTAG2, W6 to JTAG3, W7 to JTAG4, W8 to JTAG5, W9 to JTAG6, W1 to P0.0, W2 to P0.1, W3 to PWM1
Connections:
- net SD_MOSI: now also R43.2
- net SD_SCK: no longer R43.2
- net at IC7.52 (P2.11/EINT1N/I2STX_CLK): no longer PWM1.1
- net DIR5: no longer names the net of IC7.50 (P2.13/EINT3N/I2STX_SDA)
- net EN1: no longer names the net of IC7.81 (P0.4/I2SRX_CLK/CAN_RX2/CAP2.0)
- net EN2: no longer names the net of IC7.48 (P0.10/TXD2/SDA2/MAT3.0)
- net EN3: no longer names the net of IC7.59 (P0.19/DSR1/MCICLK/SDA1)
- net EN4: no longer names the net of IC7.57 (P0.21/RI1/CAN_RX1)
- net P2.7: no longer names the net of IC7.66 (P2.7/CAN_RX2/RTS1)
- net P2.8: no longer names the net of IC7.65 (P2.8/CAN_tx2/TXD2)
- net P4.29: no longer names the net of IC7.85 (P4.29/TX_MCLK/MAT2.1/RXD3)
- net PWM1: no longer names the net of IC7.68 (P2.5/PWM1.6/DTR1/TRACEDATA0)
- net PWM1: now also PWM1.1
- no-connect marks 18 -> 27
Other:
- moved on the sheet: C36, C37, JTAG1, JTAG2, JTAG3, JTAG4, JTAG5, JTAG6, PWM1, X1

Commit message: Diagram done, routing in progress.
Parts:
- added unit 4 of IC3
- added W1: TEST_1P, lpcsaur2:TP_0805, symbol TEST_1P
- C1, C10, C11, C12, C13, C14, C15, C2, C29, C3, C4, C5, C6, C7, C8, C9: footprint (none) -> Capacitors_SMD:C_0805
- C16, C17, C28, C33: footprint (none) -> Capacitors_Tantalum_SMD:TantalC_SizeD_EIA-7343_Reflow
- C18, C19: footprint (none) -> Capacitors_SMD:C_0603
- C20, C21, C22, C23, C24, C25, C26, C27: footprint ~ -> Capacitors_SMD:C_0603_HandSoldering
- C30, C31, C32: footprint ~ -> Capacitors_SMD:C_0805
- C34, C35: footprint (none) -> Capacitors_SMD:c_elec_6.3x7.7
- C36, C37: footprint ~ -> Capacitors_SMD:C_0603
- D1, D2: footprint (none) -> Diodes_ThroughHole:Diode_DO-41_SOD81_Vertical_KathodeUp
- D3, D4: footprint (none) -> Diodes_SMD:SMA_Standard
- IC1, IC2, IC3, IC4, IC5: footprint (none) -> SMD_Packages:SOIC-14_N
- IC6: footprint SOT89-3 -> TO_SOT_Packages_SMD:SOT-223
- IC7: footprint ~ -> Housings_QFP:TQFP-100_14x14mm_Pitch0.5mm
- J1, J17, J2, J28, J3, J6: footprint (none) -> Connectors_JST:JST_PH_B2B-PH-K_02x2.00mm_Straight
- J10, J23, J7, J8, J9: footprint (none) -> Connectors_JST:JST_PH_B4B-PH-K_04x2.00mm_Straight
- J11, J12, J13, J14, J15, J16, J22: footprint (none) -> Connectors_JST:JST_PH_B3B-PH-K_03x2.00mm_Straight
- J18, J20: footprint (none) -> Socket_Strips:Socket_Strip_Straight_1x03
- J19: value RELAY1 -> RELAY2; footprint (none) -> Connectors_JST:JST_PH_B2B-PH-K_02x2.00mm_Straight
- J21: footprint (none) -> Connect:USB_B
- J24, J25, J26: footprint (none) -> Terminal_Blocks:TerminalBlock_WAGO-804_RM5mm_2pol
- J27: footprint (none) -> Connectors_JST:JST_PH_B10B-PH-K_10x2.00mm_Straight
- J29: footprint (none) -> lpcsaur2:Conn_uSDcard
- J4: renamed from Y2; value Z1 -> Y2; footprint (none) -> Connectors_JST:JST_PH_B2B-PH-K_02x2.00mm_Straight
- J5: value Z2 -> Z1; footprint (none) -> Connectors_JST:JST_PH_B2B-PH-K_02x2.00mm_Straight
- JTAG1, JTAG2, JTAG3, JTAG4, JTAG5, JTAG6, P0.0, P0.1, PWM1: footprint (none) -> lpcsaur2:TP_Oblong
- L1, R33, R34, R35, R36, R37, R38, R39, R40, R42, R43, R44: footprint ~ -> Resistors_SMD:R_0603
- LED1, LED2, LED3, LED4, LED8: footprint ~ -> LEDs:LED_0603
- LED10, LED11, LED5, LED6, LED7, LED9: footprint (none) -> LEDs:LED_0603
- Q1, Q2: footprint (none) -> lpcsaur:SOT-223-3
- Q3, Q4: footprint TO-220 -> lpcsaur:SSOP-6-3; symbol MOSFET -> MOSFET-RESCUE-lpcsaur
- R1, R10, R11, R12, R13, R14, R15, R16, R19, R2, R20, R21, R22, R23, R24, R25, R26, R27, R28, R29, R3, R30, R31, R32, R4, R41, R45, R46, R5, R6, R7, R8, R9: footprint (none) -> Resistors_SMD:R_0603
- R17, R18: value 360 -> 100; footprint (none) -> Resistors_SMD:R_0603
- SW1, SW3: footprint (none) -> lpcsaur2:TactileSwitch
- SW2: footprint (none) -> lpcsaur2:TactileSwitchUpright
- X1: footprint (none) -> lpcsaur2:CrystalSmd2.5x3.2
Connections:
- net +3V3: now also Q3.S; no longer Q3.3 (S)
- net +5V: now also Q4.S, IC3.12 (4A), IC3.13 (4B); no longer Q4.3 (S)
- net GND: now also W1.1
- net P1.0: now also Q4.G; no longer Q4.1 (G)
- net P2.9: now also Q3.G; no longer Q3.1 (G)
- net P0.19: now reaches IC7.59 (P0.19/DSR1/MCICLK/SDA1)
- net P0.19: now also IC5.13 (6A)
- net P0.18: now reaches IC7.60 (P0.18/DCD1/MOSI0/MOSI)
- net P0.18: now also IC5.11 (5A)
- net P0.17: now reaches IC7.61 (P0.17/CTS1/MISO0/MISO)
- net P0.17: now also IC5.9 (4A)
- net P0.16: now reaches IC7.63 (P0.16/RXD1/SSEL0/SSEL)
- net P0.16: now also IC5.5 (3A)
- net at R32.1: now also Q3.D; no longer Q3.2 (D)
- net at J22.3 (P3): now also Q4.D; no longer Q4.2 (D)
- removed net P?: IC5.11 (5A), IC5.13 (6A), IC5.5 (3A), IC5.9 (4A)
- no-connect marks 27 -> 22
Other:
- moved on the sheet: C30, C31

Commit message: Fix 7410 footprint.
Parts:
- IC2: footprint SMD_Packages:SOIC-14_N -> SMD_Packages:SSOP-14
Changed lines of the file:
@@
 F 0 "IC2" H 16400 4850 60  0000 C CNN
 F 1 "74LV10" H 16600 5050 60  0000 C CNN
-F 2 "SMD_Packages:SOIC-14_N" H 16400 4850 60  0001 C CNN
+F 2 "SMD_Packages:SSOP-14" H 16400 4850 60  0001 C CNN
 F 3 "" H 16400 4850 60  0000 C CNN
 	1    16400 4850
@@
 F 0 "IC2" H 17100 4850 60  0000 C CNN
 F 1 "74LV10" H 17300 5050 60  0000 C CNN
-F 2 "SMD_Packages:SOIC-14_N" H 17100 4850 60  0001 C CNN
+F 2 "SMD_Packages:SSOP-14" H 17100 4850 60  0001 C CNN
 F 3 "" H 17100 4850 60  0000 C CNN
 	2    17100 4850
@@
 F 0 "IC2" H 17800 4850 60  0000 C CNN
 F 1 "74LV10" H 18000 5050 60  0000 C CNN
-F 2 "SMD_Packages:SOIC-14_N" H 17800 4850 60  0001 C CNN
+F 2 "SMD_Packages:SSOP-14" H 17800 4850 60  0001 C CNN
 F 3 "" H 17800 4850 60  0000 C CNN
 	3    17800 4850

Commit message: Complete routing.
Parts:
- removed P0.0, P0.1: TEST_1P, lpcsaur2:TP_Oblong, symbol TEST_1P
Connections:
- no-connect marks 22 -> 24
Changed lines of the file:
@@
 $EndComp
 $Comp
-L TEST_1P P0.0
-U 1 1 5756903B
-P 5350 1100
-F 0 "P0.0" V 5350 1370 50  0000 C CNN
-F 1 "TEST_1P" H 5350 1300 50  0001 C CNN
-F 2 "lpcsaur2:TP_Oblong" H 5550 1100 50  0001 C CNN
-F 3 "" H 5550 1100 50  0000 C CNN
-	1    5350 1100
-	0    -1   -1   0
-$EndComp
-$Comp
-L TEST_1P P0.1
-U 1 1 57569112
-P 5350 1200
-F 0 "P0.1" V 5350 1470 50  0000 C CNN
-F 1 "TEST_1P" H 5350 1400 50  0001 C CNN
-F 2 "lpcsaur2:TP_Oblong" H 5550 1200 50  0001 C CNN
-F 3 "" H 5550 1200 50  0000 C CNN
-	1    5350 1200
-	0    -1   -1   0
-$EndComp
-$Comp
 L USB_B J21
 U 1 1 57569989
@@
 Text GLabel 5350 2700 0    39   Input ~ 0
 P0.19
+NoConn ~ 5350 1100
+NoConn ~ 5350 1200
 $EndSCHEMATC

Commit message: Rename 10x10 to lpcsaur; delete original lpcsaur folder.
Parts:
- D1, D2: footprint Diodes_ThroughHole:Diode_DO-41_SOD81_Vertical_KathodeUp -> Diodes_SMD:DO-214AB
Changed lines of the file:
@@
 F 0 "D1" H 8550 10550 50  0000 C CNN
 F 1 "1N5822" H 8550 10350 50  0000 C CNN
-F 2 "Diodes_ThroughHole:Diode_DO-41_SOD81_Vertical_KathodeUp" H 8550 10450 50  0001 C CNN
+F 2 "Diodes_SMD:DO-214AB" H 8550 10450 50  0001 C CNN
 F 3 "" H 8550 10450 50  0000 C CNN
 	1    8550 10450
@@
 F 0 "D2" H 10800 10550 50  0000 C CNN
 F 1 "1N5822" H 10800 10350 50  0000 C CNN
-F 2 "Diodes_ThroughHole:Diode_DO-41_SOD81_Vertical_KathodeUp" H 10800 10450 50  0001 C CNN
+F 2 "Diodes_SMD:DO-214AB" H 10800 10450 50  0001 C CNN
 F 3 "" H 10800 10450 50  0000 C CNN
 	1    10800 10450

Commit message: Fix footprint for Q3, Q4.
Parts:
- Q3, Q4: footprint lpcsaur:SSOP-6-3 -> TO_SOT_Packages_SMD:TSOP-6-DGS
Changed lines of the file:
@@
 F 0 "Q3" H 2100 1325 50  0000 L CNN
 F 1 "BSL207SP" H 2100 1250 50  0000 L CNN
-F 2 "lpcsaur:SSOP-6-3" H 2100 1175 50  0001 L CIN
+F 2 "TO_SOT_Packages_SMD:TSOP-6-DGS" H 2100 1175 50  0001 L CIN
 F 3 "" H 1850 1250 50  0000 L CNN
 	1    1850 1250
@@
 F 0 "Q4" H 1750 3025 50  0000 L CNN
 F 1 "BSL207SP" H 1750 2950 50  0000 L CNN
-F 2 "lpcsaur:SSOP-6-3" H 1750 2875 50  0001 L CIN
+F 2 "TO_SOT_Packages_SMD:TSOP-6-DGS" H 1750 2875 50  0001 L CIN
 F 3 "" H 1500 2950 50  0000 L CNN
 	1    1500 2950
