File: pcb/mkssbase/mkssbase.sch (KiCad schematic (older format))
At the start: 26 parts, among them IC1 74LV11, IC2 74HCT08, J1 DOOR1, J2 DOOR2, J3 CHILLER, J4 TO_J8, J6 Conn_02x04_Odd_Even, J7 LASER_AUX, J8 LASER

Commit message: Fix footprints.
Parts:
- C1, C2, C3, C4, C5, C6: footprint Capacitors_SMD:C_0805 -> Capacitor_SMD:C_0805_2012Metric
- IC1, IC2: footprint (none) -> Package_SO:SOIC-14_3.9x8.7mm_P1.27mm
- J1, J2: footprint Connectors_JST:JST_PH_B3B-PH-K_03x2.00mm_Straight -> Connector_JST:JST_PH_B3B-PH-K_1x03_P2.00mm_Vertical
- J3: footprint Connectors_JST:JST_PH_B2B-PH-K_02x2.00mm_Straight -> Connector_JST:JST_PH_B2B-PH-K_1x02_P2.00mm_Vertical
- J4: footprint Connectors:PINHEAD1-6 -> Connector_JST:JST_XH_B06B-XH-A_1x06_P2.50mm_Vertical
- J6: footprint (none) -> Connector_PinSocket_2.54mm:PinSocket_2x04_P2.54mm_Vertical
- J7, J8: footprint Connectors_JST:JST_PH_B4B-PH-K_04x2.00mm_Straight -> Connector_JST:JST_PH_B4B-PH-K_1x04_P2.00mm_Vertical
- LED1: footprint LEDs:LED_0603 -> LED_SMD:LED_0603_1608Metric
- R1, R2, R3, R4, R5, R6, R7, R8, R9: footprint Resistors_SMD:R_0603 -> Resistor_SMD:R_0603_1608Metric
- R13: footprint (none) -> Resistor_SMD:R_0603_1608Metric
Changed lines of the file:
@@
 F 0 "IC1" H 4950 4550 60  0000 C CNN
 F 1 "74LV11" H 5150 4750 60  0000 C CNN
-F 2 "" H 4950 4550 60  0001 C CNN
+F 2 "Package_SO:SOIC-14_3.9x8.7mm_P1.27mm" H 4950 4550 60  0001 C CNN
 F 3 "http://www.ti.com/lit/gpn/sn74LS11" H 4950 4550 60  0001 C CNN
 	2    4950 4550
@@
 F 0 "R3" V 2980 5000 50  0000 C CNN
 F 1 "1K" V 2900 5000 50  0000 C CNN
-F 2 "Resistors_SMD:R_0603" V 2830 5000 50  0001 C CNN
+F 2 "Resistor_SMD:R_0603_1608Metric" V 2830 5000 50  0001 C CNN
 F 3 "" H 2900 5000 50  0000 C CNN
 	1    2900 5000
@@
 F 0 "R4" V 3280 5000 50  0000 C CNN
 F 1 "1K" V 3200 5000 50  0000 C CNN
-F 2 "Resistors_SMD:R_0603" V 3130 5000 50  0001 C CNN
+F 2 "Resistor_SMD:R_0603_1608Metric" V 3130 5000 50  0001 C CNN
 F 3 "" H 3200 5000 50  0000 C CNN
 	1    3200 5000
@@
 F 0 "J3" V 3100 2850 50  0000 C CNN
 F 1 "CHILLER" H 3000 2650 50  0000 C CNN
-F 2 "Connectors_JST:JST_PH_B2B-PH-K_02x2.00mm_Straight" H 2950 2850 50  0001 C CNN
+F 2 "Connector_JST:JST_PH_B2B-PH-K_1x02_P2.00mm_Vertical" H 2950 2850 50  0001 C CNN
 F 3 "" H 2950 2850 50  0000 C CNN
 	1    2950 2850
@@
 F 0 "R5" V 3680 3150 50  0000 C CNN
 F 1 "1K" V 3600 3150 50  0000 C CNN
-F 2 "Resistors_SMD:R_0603" V 3530 3150 50  0001 C CNN
+F 2 "Resistor_SMD:R_0603_1608Metric" V 3530 3150 50  0001 C CNN
 F 3 "" H 3600 3150 50  0000 C CNN
 	1    3600 3150
@@
 F 0 "R9" V 8630 3950 50  0000 C CNN
 F 1 "1K" V 8550 3950 50  0000 C CNN
-F 2 "Resistors_SMD:R_0603" V 8480 3950 50  0001 C CNN
+F 2 "Resistor_SMD:R_0603_1608Metric" V 8480 3950 50  0001 C CNN
 F 3 "" H 8550 3950 50  0000 C CNN
 	1    8550 3950
@@
 F 0 "LED1" H 8550 4500 50  0000 C CNN
 F 1 "Disable" H 8550 4300 50  0000 C CNN
-F 2 "LEDs:LED_0603" H 8550 4400 50  0001 C CNN
+F 2 "LED_SMD:LED_0603_1608Metric" H 8550 4400 50  0001 C CNN
 F 3 "" H 8550 4400 50  0000 C CNN
 	1    8550 4400
@@
 F 0 "C4" H 625 2950 50  0000 L CNN
 F 1 "100n" H 625 2750 50  0000 L CNN
-F 2 "Capacitors_SMD:C_0805" H 638 2700 50  0001 C CNN
+F 2 "Capacitor_SMD:C_0805_2012Metric" H 638 2700 50  0001 C CNN
 F 3 "" H 600 2850 50  0000 C CNN
 	1    600  2850
@@
 F 0 "IC2" H 7750 3650 60  0000 C CNN
 F 1 "74HCT08" H 7850 3550 60  0000 C CNN
-F 2 "" H 7650 3350 60  0001 C CNN
+F 2 "Package_SO:SOIC-14_3.9x8.7mm_P1.27mm" H 7650 3350 60  0001 C CNN
 F 3 "http://www.ti.com/lit/gpn/sn74LS08" H 7650 3350 60  0001 C CNN
 	1    7650 3350
@@
 F 0 "IC2" H 7750 4450 60  0000 C CNN
 F 1 "74HCT08" H 7850 4350 60  0000 C CNN
-F 2 "" H 7650 4150 60  0001 C CNN
+F 2 "Package_SO:SOIC-14_3.9x8.7mm_P1.27mm" H 7650 4150 60  0001 C CNN
 F 3 "http://www.ti.com/lit/gpn/sn74LS08" H 7650 4150 60  0001 C CNN
 	2    7650 4150
@@
 F 0 "R6" V 3700 4550 50  0000 C CNN
 F 1 "5K6" V 3800 4550 50  0000 C CNN
-F 2 "Resistors_SMD:R_0603" V 3730 4550 50  0001 C CNN
+F 2 "Resistor_SMD:R_0603_1608Metric" V 3730 4550 50  0001 C CNN
 F 3 "" H 3800 4550 50  0000 C CNN
 	1    3800 4550
@@
 F 0 "R7" V 3880 4650 50  0000 C CNN
 F 1 "5K6" V 3800 4650 50  0000 C CNN
-F 2 "Resistors_SMD:R_0603" V 3730 4650 50  0001 C CNN
+F 2 "Resistor_SMD:R_0603_1608Metric" V 3730 4650 50  0001 C CNN
 F 3 "" H 3800 4650 50  0000 C CNN
 	1    3800 4650
@@
 F 0 "C3" H 4625 5100 50  0000 L CNN
 F 1 "100n" H 4625 4900 50  0000 L CNN
-F 2 "Capacitors_SMD:C_0805" H 4638 4850 50  0001 C CNN
+F 2 "Capacitor_SMD:C_0805_2012Metric" H 4638 4850 50  0001 C CNN
 F 3 "" H 4600 5000 50  0000 C CNN
 	1    4600 5000
@@
 F 0 "C2" H 4375 5100 50  0000 L CNN
 F 1 "100n" H 4375 4900 50  0000 L CNN
-F 2 "Capacitors_SMD:C_0805" H 4388 4850 50  0001 C CNN
+F 2 "Capacitor_SMD:C_0805_2012Metric" H 4388 4850 50  0001 C CNN
 F 3 "" H 4350 5000 50  0000 C CNN
 	1    4350 5000
@@
 F 0 "R1" V 2050 4700 50  0000 C CNN
 F 1 "100" V 2150 4650 50  0000 C CNN
-F 2 "Resistors_SMD:R_0603" V 2080 4650 50  0001 C CNN
+F 2 "Resistor_SMD:R_0603_1608Metric" V 2080 4650 50  0001 C CNN
 F 3 "" H 2150 4650 50  0000 C CNN
 	1    2150 4650
@@
 F 0 "R2" V 2050 5500 50  0000 C CNN
 F 1 "100" V 2150 5450 50  0000 C CNN
-F 2 "Resistors_SMD:R_0603" V 2080 5450 50  0001 C CNN
+F 2 "Resistor_SMD:R_0603_1608Metric" V 2080 5450 50  0001 C CNN
 F 3 "" H 2150 5450 50  0000 C CNN
 	1    2150 5450
@@
 F 0 "C5" H 2475 2950 50  0000 L CNN
 F 1 "100n" H 2475 2750 50  0000 L CNN
-F 2 "Capacitors_SMD:C_0805" H 2488 2700 50  0001 C CNN
+F 2 "Capacitor_SMD:C_0805_2012Metric" H 2488 2700 50  0001 C CNN
 F 3 "" H 2450 2850 50  0000 C CNN
 	1    2450 2850
@@
 F 0 "J8" H 9300 3600 50  0000 C CNN
 F 1 "LASER" V 9400 3350 50  0000 C CNN
-F 2 "Connectors_JST:JST_PH_B4B-PH-K_04x2.00mm_Straight" H 9300 3350 50  0001 C CNN
+F 2 "Connector_JST:JST_PH_B4B-PH-K_1x04_P2.00mm_Vertical" H 9300 3350 50  0001 C CNN
 F 3 "" H 9300 3350 50  0000 C CNN
 	1    9300 3350
@@
 F 0 "C1" H 4125 3250 50  0000 L CNN
 F 1 "100n" H 4125 3050 50  0000 L CNN
-F 2 "Capacitors_SMD:C_0805" H 4138 3000 50  0001 C CNN
+F 2 "Capacitor_SMD:C_0805_2012Metric" H 4138 3000 50  0001 C CNN
 F 3 "" H 4100 3150 50  0000 C CNN
 	1    4100 3150
@@
 F 0 "R8" V 3930 2950 50  0000 C CNN
 F 1 "5K6" V 3850 2950 50  0000 C CNN
-F 2 "Resistors_SMD:R_0603" V 3780 2950 50  0001 C CNN
+F 2 "Resistor_SMD:R_0603_1608Metric" V 3780 2950 50  0001 C CNN
 F 3 "" H 3850 2950 50  0000 C CNN
 	1    3850 2950
@@
 F 0 "IC2" H 6600 5650 60  0000 C CNN
 F 1 "74HCT08" H 6700 5550 60  0000 C CNN
-F 2 "" H 6500 5350 60  0001 C CNN
+F 2 "Package_SO:SOIC-14_3.9x8.7mm_P1.27mm" H 6500 5350 60  0001 C CNN
 F 3 "http://www.ti.com/lit/gpn/sn74LS08" H 6500 5350 60  0001 C CNN
 	3    6500 5350
@@
 F 0 "J1" H 1700 4750 50  0000 C CNN
 F 1 "DOOR1" H 1950 4550 50  0000 C CNN
-F 2 "Connectors_JST:JST_PH_B3B-PH-K_03x2.00mm_Straight" H 1700 4550 50  0001 C CNN
+F 2 "Connector_JST:JST_PH_B3B-PH-K_1x03_P2.00mm_Vertical" H 1700 4550 50  0001 C CNN
 F 3 "" H 1700 4550 50  0001 C CNN
 	1    1700 4550
@@
 F 0 "J2" H 1700 5550 50  0000 C CNN
 F 1 "DOOR2" H 1950 5350 50  0000 C CNN
-F 2 "Connectors_JST:JST_PH_B3B-PH-K_03x2.00mm_Straight" H 1700 5350 50  0001 C CNN
+F 2 "Connector_JST:JST_PH_B3B-PH-K_1x03_P2.00mm_Vertical" H 1700 5350 50  0001 C CNN
 F 3 "" H 1700 5350 50  0001 C CNN
 	1    1700 5350
@@
 F 0 "IC1" H 5900 3750 60  0000 C CNN
 F 1 "74LV11" H 6000 3650 60  0000 C CNN
-F 2 "" H 5800 3450 60  0001 C CNN
+F 2 "Package_SO:SOIC-14_3.9x8.7mm_P1.27mm" H 5800 3450 60  0001 C CNN
 F 3 "http://www.ti.com/lit/gpn/sn74LS11" H 5800 3450 60  0001 C CNN
 	1    5800 3450
@@
 F 0 "IC2" H 6600 6350 60  0000 C CNN
 F 1 "74HCT08" H 6700 6250 60  0000 C CNN
-F 2 "" H 6500 6050 60  0001 C CNN
+F 2 "Package_SO:SOIC-14_3.9x8.7mm_P1.27mm" H 6500 6050 60  0001 C CNN
 F 3 "http://www.ti.com/lit/gpn/sn74LS08" H 6500 6050 60  0001 C CNN
 	4    6500 6050
@@
 F 0 "J7" H 9300 2550 50  0000 C CNN
 F 1 "LASER_AUX" V 9400 2300 50  0000 C CNN
-F 2 "Connectors_JST:JST_PH_B4B-PH-K_04x2.00mm_Straight" H 9300 2300 50  0001 C CNN
+F 2 "Connector_JST:JST_PH_B4B-PH-K_1x04_P2.00mm_Vertical" H 9300 2300 50  0001 C CNN
 F 3 "" H 9300 2300 50  0001 C CNN
 	1    9300 2300
@@
 F 0 "C6" H 7625 1100 50  0000 L CNN
 F 1 "100n" H 7625 900 50  0000 L CNN
-F 2 "Capacitors_SMD:C_0805" H 7638 850 50  0001 C CNN
+F 2 "Capacitor_SMD:C_0805_2012Metric" H 7638 850 50  0001 C CNN
 F 3 "" H 7600 1000 50  0001 C CNN
 	1    7600 1000
@@
 F 0 "IC1" H 3900 6250 60  0000 C CNN
 F 1 "74LV11" H 4000 6150 60  0000 C CNN
-F 2 "" H 3800 5950 60  0001 C CNN
+F 2 "Package_SO:SOIC-14_3.9x8.7mm_P1.27mm" H 3800 5950 60  0001 C CNN
 F 3 "http://www.ti.com/lit/gpn/sn74LS11" H 3800 5950 60  0001 C CNN
 	3    3800 5950
@@
 F 0 "J4" H 4650 1500 50  0000 C CNN
 F 1 "TO_J8" V 4750 1150 50  0000 C CNN
-F 2 "Connectors:PINHEAD1-6" H 4650 1150 50  0001 C CNN
+F 2 "Connector_JST:JST_XH_B06B-XH-A_1x06_P2.50mm_Vertical" H 4650 1150 50  0001 C CNN
 F 3 "" H 4650 1150 50  0001 C CNN
 	1    4650 1150
@@
 F 0 "R13" H 7270 4596 50  0000 L CNN
 F 1 "10K" H 7270 4505 50  0000 L CNN
-F 2 "" V 7130 4550 50  0001 C CNN
+F 2 "Resistor_SMD:R_0603_1608Metric" V 7130 4550 50  0001 C CNN
 F 3 "" H 7200 4550 50  0001 C CNN
 	1    7200 4550
@@
 F 0 "J6" H 8250 1567 50  0000 C CNN
 F 1 "Conn_02x04_Odd_Even" H 8250 1476 50  0000 C CNN
-F 2 "" H 8200 1250 50  0001 C CNN
+F 2 "Connector_PinSocket_2.54mm:PinSocket_2x04_P2.54mm_Vertical" H 8200 1250 50  0001 C CNN
 F 3 "~" H 8200 1250 50  0001 C CNN
 	1    8200 1250
@@
 F 0 "IC2" H 1980 2896 50  0000 L CNN
 F 1 "74HCT08" H 1980 2805 50  0000 L CNN
-F 2 "" H 1750 2850 50  0001 C CNN
+F 2 "Package_SO:SOIC-14_3.9x8.7mm_P1.27mm" H 1750 2850 50  0001 C CNN
 F 3 "http://www.ti.com/lit/gpn/sn74LS08" H 1750 2850 50  0001 C CNN
 	5    1750 2850
@@
 F 0 "IC1" H 1280 2896 50  0000 L CNN
 F 1 "74LV11" H 1280 2805 50  0000 L CNN
-F 2 "" H 1050 2850 50  0001 C CNN
+F 2 "Package_SO:SOIC-14_3.9x8.7mm_P1.27mm" H 1050 2850 50  0001 C CNN
 F 3 "http://www.ti.com/lit/gpn/sn74LS11" H 1050 2850 50  0001 C CNN
 	4    1050 2850

Commit message: Add chiller control.
Parts:
- LED1: value Disable -> Enable
Changed lines of the file:
@@
 EESchema Schematic File Version 4
 LIBS:mkssbase-cache
+LIBS:chillercontrol-cache
 EELAYER 26 0
 EELAYER END
 $Descr A4 11693 8268
 encoding utf-8
-Sheet 1 2
+Sheet 1 3
 Title ""
 Date ""
@@
 P 8550 4400
 F 0 "LED1" H 8550 4500 50  0000 C CNN
-F 1 "Disable" H 8550 4300 50  0000 C CNN
+F 1 "Enable" V 8500 4100 50  0000 C CNN
 F 2 "LED_SMD:LED_0603_1608Metric" H 8550 4400 50  0001 C CNN
 F 3 "" H 8550 4400 50  0000 C CNN
@@
 	1    0    0    -1
 $EndComp
+$Sheet
+S 850  6850 1550 500
+U 5C787D7D
+F0 "chillercontrol" 60
+F1 "chillercontrol.sch" 60
+$EndSheet
 $EndSCHEMATC

Commit message: Fix wrong supply voltage to IC1.
Connections:
- net +3V3: now also C4.1, IC1.14 (VCC)
- net +5V: no longer C4.1, IC1.14 (VCC)
Changed lines of the file:
@@
 $EndComp
-Wire Wire Line
-	1750 2350 1050 2350
 Wire Wire Line
 	1050 3350 1050 3400
@@
 Wire Wire Line
 	1750 3400 2450 3400
-Connection ~ 1050 2350
 Wire Wire Line
 	600  3000 600  3400
@@
 F1 "chillercontrol.sch" 60
 $EndSheet
+$Comp
+L power:+3V3 #PWR?
+U 1 1 5C8E6364
+P 1050 2250
+F 0 "#PWR?" H 1050 2100 50  0001 C CNN
+F 1 "+3V3" H 1065 2423 50  0000 C CNN
+F 2 "" H 1050 2250 50  0001 C CNN
+F 3 "" H 1050 2250 50  0001 C CNN
+	1    1050 2250
+	1    0    0    -1
+$EndComp
+Wire Wire Line
+	1050 2250 1050 2350
+Connection ~ 1050 2350
 $EndSCHEMATC

Commit message: Add inverted laser control signal.
Parts:
- removed J7: LASER_AUX, Connector_JST:JST_PH_B4B-PH-K_1x04_P2.00mm_Vertical, symbol Connector_Generic:Conn_01x04
- removed J8: LASER, Connector_JST:JST_PH_B4B-PH-K_1x04_P2.00mm_Vertical, symbol Connector_Generic:Conn_01x04
- added C12: 100n, Capacitor_SMD:C_0603_1608Metric, symbol Device:C
- added IC5: 74HCT04, Package_SO:SOIC-14_3.9x8.7mm_P1.27mm, symbol 74xx:74HCT04
- added J7: LASER_AUX, Connector_JST:JST_PH_B5B-PH-K_1x05_P2.00mm_Vertical, symbol Connector_Generic:Conn_01x05
- added J8: LASER, Connector_JST:JST_PH_B5B-PH-K_1x05_P2.00mm_Vertical, symbol Connector_Generic:Conn_01x05
- C1, C2, C3, C4, C5, C6: footprint Capacitor_SMD:C_0805_2012Metric -> Capacitor_SMD:C_0603_1608Metric
Connections:
- net +5V: now also C12.1, IC5.11, IC5.13, IC5.14 (VCC), IC5.9, J7.1 (Pin_1), J8.1 (Pin_1)
- net GND: now also C12.2, IC5.3, IC5.5, IC5.7 (GND), J7.5 (Pin_5), J8.5 (Pin_5)
- net at IC2.3, R9.1: now also IC5.1, J7.3 (Pin_3), J8.3 (Pin_3)
- net at IC2.6: now also J7.4 (Pin_4), J8.4 (Pin_4)
- new net: IC5.2, J7.2 (Pin_2), J8.2 (Pin_2)
- no-connect marks 7 -> 12
Other:
- note added: "1: +5V\n2: TL\n3: TH\n4: PWM\n5: GND"
- note removed: "1: +5V\n2: TH\n3: PWM\n4: GND"
- moved on the sheet: C4, C5, IC1C, IC1D, IC2E
