File: pcb/counter/counter.kicad_pcb (KiCad board)
At the start: 2 copper layers, 85.9 x 60.5 mm, 15 parts, among them J1 Conn_01x01, J2 Conn_01x01, J3 Conn_01x01, J4 Conn_01x06, J5 Conn_01x02, J6 Conn_01x05, Q1 Q_NPN_CBE, U1 74LS08

Commit message: Fix track widths, outline.
Parts:
- added J7: Conn_01x03, TerminalBlock:TerminalBlock_Altech_AK300-3_P5.00mm, F.Cu at (71.6, 74.7)
- added R4: 100k, Resistor_THT:R_Axial_DIN0411_L9.9mm_D3.6mm_P7.62mm_Vertical, F.Cu at (116.8, 42.7)
- R3: value R -> 1k
- U1: value 74LS08 -> 74HC08
- moved J5 20.2 mm to (69.1, 49.8), turned to 270 degrees
Connections:
- U1 pad 1: Net-(J4-Pad3) -> Net-(J4-Pad2)
- U1 pad 2: Net-(J4-Pad3) -> Net-(J4-Pad2)
Routing:
- net Net-(J3-Pad1): track 100.3 -> 69.6 mm
- net Net-(J4-Pad2): track 10.7 -> 39.2 mm
- net Net-(J4-Pad3): track 35.6 -> 13.0 mm
- net Net-(J2-Pad1): track 21.2 -> 39.5 mm
- net GND: track 134.3 -> 151.5 mm
- net Net-(J1-Pad1): track 0.00 -> 11.1 mm
- net +5V: track 126.1 -> 130.9 mm
- net Net-(J5-Pad1): track 19.3 -> 16.4 mm
Other:
- board size 85.9 x 60.5 mm -> 91.4 x 51.8 mm

Commit message: Fix error.
Connections:
- R4 pad 1: Net-(J4-Pad2) -> Net-(J4-Pad1)
- U1 pad 1: Net-(J4-Pad2) -> Net-(J4-Pad1)
- U1 pad 2: Net-(J4-Pad2) -> Net-(J4-Pad1)
Routing:
- net Net-(J4-Pad1): track 9.67 -> 39.2 mm
- net Net-(J4-Pad2): track 39.2 -> 10.7 mm
- net Net-(J3-Pad1): track 69.6 -> 68.6 mm
Changed lines of the file:
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@@
     (thickness 1.6)
     (drawings 4)
-    (tracks 116)
+    (tracks 115)
     (zones 0)
     (modules 17)
@@
   )
   (setup
-    (last_trace_width 0.25)
+    (last_trace_width 2)
     (user_trace_width 0.5)
     (user_trace_width 1)
@@
     )
     (pad 1 thru_hole rect (at 0 0 90) (size 2.4 1.6) (drill 0.8) (layers *.Cu *.Mask)
-      (net 8 "Net-(J4-Pad2)"))
+      (net 10 "Net-(J4-Pad1)"))
     (pad 8 thru_hole oval (at 7.62 15.24 90) (size 2.4 1.6) (drill 0.8) (layers *.Cu *.Mask)
       (net 17 "Net-(U1-Pad8)"))
     (pad 2 thru_hole oval (at 0 2.54 90) (size 2.4 1.6) (drill 0.8) (layers *.Cu *.Mask)
-      (net 8 "Net-(J4-Pad2)"))
+      (net 10 "Net-(J4-Pad1)"))
     (pad 9 thru_hole oval (at 7.62 12.7 90) (size 2.4 1.6) (drill 0.8) (layers *.Cu *.Mask)
       (net 2 GND))
@@
     )
     (pad 1 thru_hole circle (at 0 0 90) (size 2.4 2.4) (drill 1.2) (layers *.Cu *.Mask)
-      (net 8 "Net-(J4-Pad2)"))
+      (net 10 "Net-(J4-Pad1)"))
     (pad 2 thru_hole oval (at 7.62 0 90) (size 2.4 2.4) (drill 1.2) (layers *.Cu *.Mask)
       (net 2 GND))
@@
   (segment (start 89.916 53.848) (end 89.916 69.596) (width 2) (layer B.Cu) (net 6))
   (segment (start 89.916 69.596) (end 89.916 74.916) (width 2) (layer B.Cu) (net 6))
-  (segment (start 97.5 79.284) (end 97.5 75) (width 2) (layer B.Cu) (net 7))
-  (segment (start 67.564 82.804) (end 93.98 82.804) (width 2) (layer B.Cu) (net 7))
-  (segment (start 65.74901 80.98901) (end 67.564 82.804) (width 2) (layer B.Cu) (net 7))
-  (segment (start 93.98 82.804) (end 97.5 79.284) (width 2) (layer B.Cu) (net 7))
-  (segment (start 68.648 64.676) (end 65.76 67.564) (width 2) (layer B.Cu) (net 7))
-  (segment (start 71.628 64.676) (end 68.648 64.676) (width 1) (layer B.Cu) (net 7))
   (segment (start 65.76 67.844) (end 65.74901 67.85499) (width 1) (layer B.Cu) (net 7))
-  (segment (start 65.76 67.564) (end 65.76 67.844) (width 1) (layer B.Cu) (net 7))
-  (segment (start 66.04 67.85499) (end 66.04 80.98901) (width 2) (layer B.Cu) (net 7))
   (segment (start 71.628 57.404) (end 71.628 64.676) (width 1) (layer B.Cu) (net 7))
   (segment (start 69.088 54.864) (end 71.628 57.404) (width 1) (layer B.Cu) (net 7))
+  (segment (start 97.5 79.284) (end 97.5 75) (width 2) (layer B.Cu) (net 7))
+  (segment (start 69.248 64.676) (end 66.548 67.376) (width 2) (layer B.Cu) (net 7))
+  (segment (start 93.98 82.804) (end 97.5 79.284) (width 2) (layer B.Cu) (net 7))
+  (segment (start 66.548 67.376) (end 66.548 81.788) (width 2) (layer B.Cu) (net 7))
+  (segment (start 71.628 64.676) (end 69.248 64.676) (width 2) (layer B.Cu) (net 7))
+  (segment (start 66.548 81.788) (end 67.564 82.804) (width 2) (layer B.Cu) (net 7))
+  (segment (start 67.564 82.804) (end 93.98 82.804) (width 2) (layer B.Cu) (net 7))
   (segment (start 120.824 65.532) (end 120.824 68.5) (width 0.5) (layer B.Cu) (net 8))
   (segment (start 123.444 71.12) (end 123.444 75.184) (width 0.5) (layer B.Cu) (net 8))
   (segment (start 120.824 68.5) (end 123.444 71.12) (width 0.5) (layer B.Cu) (net 8))
-  (segment (start 120.904 46.228) (end 123.444 46.228) (width 0.5) (layer B.Cu) (net 8))
-  (segment (start 120.824 57.992) (end 120.824 65.532) (width 0.5) (layer B.Cu) (net 8))
-  (segment (start 123.444 46.228) (end 123.444 55.372) (width 0.5) (layer B.Cu) (net 8))
-  (segment (start 123.444 55.372) (end 120.824 57.992) (width 0.5) (layer B.Cu) (net 8))
-  (segment (start 120.396 46.228) (end 120.904 46.228) (width 0.5) (layer B.Cu) (net 8))
-  (segment (start 116.84 42.672) (end 120.396 46.228) (width 0.5) (layer B.Cu) (net 8))
+  (segment (start 120.904 46.228) (end 123.444 46.228) (width 0.5) (layer B.Cu) (net 10))
+  (segment (start 120.396 46.228) (end 120.904 46.228) (width 0.5) (layer B.Cu) (net 10))
+  (segment (start 116.84 42.672) (end 120.396 46.228) (width 0.5) (layer B.Cu) (net 10))
   (segment (start 123.324 67.532) (end 123.356 67.564) (width 0.5) (layer B.Cu) (net 9))
   (segment (start 123.324 65.532) (end 123.324 67.532) (width 0.5) (layer B.Cu) (net 9))
@@
   (segment (start 118.324 75.144) (end 118.364 75.184) (width 0.5) (layer B.Cu) (net 10))
   (segment (start 118.324 65.532) (end 118.324 75.144) (width 0.5) (layer B.Cu) (net 10))
+  (segment (start 123.444 46.228) (end 123.444 55.372) (width 0.5) (layer B.Cu) (net 10))
+  (segment (start 118.324 60.492) (end 118.324 65.532) (width 0.5) (layer B.Cu) (net 10))
+  (segment (start 123.444 55.372) (end 118.324 60.492) (width 0.5) (layer B.Cu) (net 10))
   (segment (start 138.684 75.184) (end 143.764 75.184) (width 0.5) (layer B.Cu) (net 11))
   (segment (start 82.296 51.348) (end 82.296 53.848) (width 1) (layer B.Cu) (net 12))
@@
   (segment (start 125.984 46.228) (end 125.984 59.436) (width 0.5) (layer B.Cu) (net 15))
   (segment (start 133.604 46.228) (end 133.604 50.8) (width 0.5) (layer B.Cu) (net 16))
-  (zone (net 0) (net_name "") (layer B.Cu) (hatch edge 0.508)
-    (connect_pads (clearance 0.508))
-    (min_thickness 0.254)
-    (keepout (tracks not_allowed) (vias not_allowed) (copperpour allowed))
-    (fill (arc_segments 32) (thermal_gap 0.508) (thermal_bridge_width 0.508))
-    (polygon
-      (pts
-        (xy 96.52 65.532) (xy 104.14 72.644) (xy 104.14 84.836) (xy 65.024 84.836) (xy 65.024 37.592)
-        (xy 96.52 37.592)
-      )
-    )
-  )
 )
