File: pcb/counter/counter.sch (KiCad schematic (older format))
At the start: 16 parts, among them J1 Conn_01x01, J2 Conn_01x01, J3 Conn_01x01, J4 Conn_01x06, J5 Conn_01x02, J6 Conn_01x05, Q1 Q_NPN_CBE, U1 74HC08

Commit message: Fix track widths, outline.
Parts:
- added J7: Conn_01x03, TerminalBlock:TerminalBlock_Altech_AK300-3_P5.00mm, symbol Connector_Generic:Conn_01x03
- R4: footprint (none) -> Resistor_THT:R_Axial_DIN0411_L9.9mm_D3.6mm_P7.62mm_Vertical
Connections:
- net at J3.1 (Pin_1), J5.2 (Pin_2): now also J7.3 (Pin_3)
- net at J2.1 (Pin_1), RLY1.5: now also J7.2 (Pin_2)
- net at J1.1 (Pin_1): now also J7.1 (Pin_1)
- no-connect marks 3 -> 2
Changed lines of the file:
@@
 $EndComp
 Wire Wire Line
-	1650 2050 2800 2050
+	1650 2050 2050 2050
 Wire Wire Line
 	2800 1950 2500 1950
@@
 NoConn ~ 4100 5650
 NoConn ~ 3100 5650
-NoConn ~ 1650 1750
 $Comp
 L Connector_Generic:Conn_01x01 J2
@@
 $EndComp
 Wire Wire Line
-	1650 1900 2100 1900
+	1650 1900 1950 1900
 $Comp
 L Device:R R4
@@
 F 0 "R4" H 2320 4246 50  0000 L CNN
 F 1 "100k" H 2320 4155 50  0000 L CNN
-F 2 "" V 2180 4200 50  0001 C CNN
+F 2 "Resistor_THT:R_Axial_DIN0411_L9.9mm_D3.6mm_P7.62mm_Vertical" V 2180 4200 50  0001 C CNN
 F 3 "~" H 2250 4200 50  0001 C CNN
 	1    2250 4200
@@
 	2250 3000 2800 3000
 Connection ~ 2250 3750
+$Comp
+L Connector_Generic:Conn_01x03 J7
+U 1 1 5E0A80A3
+P 1450 2450
+F 0 "J7" H 1368 2767 50  0000 C CNN
+F 1 "Conn_01x03" H 1368 2676 50  0000 C CNN
+F 2 "TerminalBlock:TerminalBlock_Altech_AK300-3_P5.00mm" H 1450 2450 50  0001 C CNN
+F 3 "~" H 1450 2450 50  0001 C CNN
+	1    1450 2450
+	-1   0    0    -1
+$EndComp
+Wire Wire Line
+	1650 1750 1850 1750
+Wire Wire Line
+	1850 1750 1850 2350
+Wire Wire Line
+	1850 2350 1650 2350
+Wire Wire Line
+	1950 1900 1950 2450
+Wire Wire Line
+	1950 2450 1650 2450
+Connection ~ 1950 1900
+Wire Wire Line
+	1950 1900 2100 1900
+Wire Wire Line
+	2050 2050 2050 2550
+Wire Wire Line
+	2050 2550 1650 2550
+Connection ~ 2050 2050
+Wire Wire Line
+	2050 2050 2800 2050
 $EndSCHEMATC

Commit message: Fix error.
Connections:
- net at J4.1 (Pin_1), J6.2 (Pin_2): now also R4.1, U1.1, U1.2
- new net: J4.2 (Pin_2), J6.3 (Pin_3)
Changed lines of the file:
@@
 $EndComp
 Wire Wire Line
-	1650 3000 2250 3000
-Wire Wire Line
-	2800 2900 1650 2900
+	2800 2900 2250 2900
 $Comp
 L power:+5V #PWR04
@@
 Wire Wire Line
 	1650 3100 2800 3100
-Wire Wire Line
-	2250 3000 2250 3750
-Connection ~ 2250 3000
-Wire Wire Line
-	2250 3000 2800 3000
 Connection ~ 2250 3750
 $Comp
@@
 Wire Wire Line
 	2050 2050 2800 2050
+Connection ~ 2250 2900
+Wire Wire Line
+	2250 2900 1650 2900
+Wire Wire Line
+	2250 2900 2250 3750
+Wire Wire Line
+	1650 3000 2800 3000
 $EndSCHEMATC
